File: UccMicroDuino/UccMicroDuino.kicad_sch (KiCad schematic)
At the start: 14 parts, among them J1 USB_PCB_A, J2 Header, U1 ATtiny85-20S

Commit message: 2621679 - Mi primer versionado en GitBash
Other:
- note added: "Circuito Principal"
- note removed: "Main Circuit"
Changed lines of the file:
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@@
 		)
 	)
-	(text "Main Circuit"
+	(text "Circuito Principal\n"
 		(exclude_from_sim no)
 		(at 55.1942 140.9954 0)
